Commit message: Added imu sensor. Fixed missing TF.

File: irobot_create_description/urdf/create3.urdf.xacro (robot description, xacro)
@@ -4,4 +4,5 @@
   <xacro:include filename="$(find irobot_create_description)/urdf/button.urdf.xacro" />
   <xacro:include filename="$(find irobot_create_description)/urdf/caster.urdf.xacro" />
+  <xacro:include filename="$(find irobot_create_description)/urdf/sensors/imu.urdf.xacro" />
   <xacro:include filename="$(find irobot_create_description)/urdf/common_properties.urdf.xacro"/>
   <xacro:include filename="$(find irobot_create_description)/urdf/wheel_with_wheeldrop.urdf.xacro" />
@@ -81,4 +82,8 @@
     </inertial>
   </xacro:bumper>
+  <!-- IMU -->
+  <xacro:imu_sensor gazebo="$(arg gazebo)" namespace="$(arg namespace)">
+    <origin xyz="0.050613 0.043673 ${0.0202 + base_link_z_offset}"/>
+  </xacro:imu_sensor>
   <!-- Wheels with mechanical wheel drop -->
   <xacro:wheel_with_wheeldrop name="left" gazebo="$(arg gazebo)" namespace="$(arg namespace)">

File: irobot_create_description/urdf/sensors/imu.urdf.xacro (robot description, xacro)
@@ -56,4 +56,7 @@
         </linear_acceleration>
       </imu>
+      <xacro:if value="${gazebo == 'ignition'}">
+        <plugin filename="gz-sim-imu-system" name="gz::sim::systems::Imu"/>
+      </xacro:if>
       <xacro:if value="${gazebo == 'classic'}">
         <plugin name="${name}_plugin" filename="libgazebo_ros_create_imu.so">
